File: Patchwork Playground.kicad_pcb (KiCad board)
At the start: 2 copper layers, 100 x 60 mm, 90 parts, among them J1 PADS, J2 USB_C_Receptacle_USB2.0, J3 PADS, J4 POGO, J5 PADS, J6 JST-GH-4P, SW1 SW_SPDT, SW2 SW_SPDT, SW3 SW_SPDT, SW4 BUTTON, SW5 SW_SPDT, SW6 SW_SPDT, SW7 SW_SPDT, U1 SMF05CT1G, U2 M3406, U3 BQ21040DBVR, U4 SMF05CT1G, U5 QMC5883L, U6 BC805M, U7 LSM6DSV

Commit message: stupid jlc order number
Other:
- board text added: "JLCJLCJLCJLC"
Changed lines of the file:
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@@
     )
+  )
+  (gr_text "JLCJLCJLCJLC" (at 153.200909 128.785418) (layer "B.SilkS")
+    (effects (font (size 1 1) (thickness 0.15)) (justify left bottom mirror))
   )
   (gr_text locked "Development board - not for consumer use" (at 185.8 100.258819) (layer "B.SilkS")
