File: Patchwork Playground.kicad_sch (KiCad schematic)
At the start: 89 parts, among them J1 PADS, J2 USB_C_Receptacle_USB2.0, J3 PADS, J4 POGO, J5 PADS, J6 JST-GH-4P, SW1 SW_SPDT, SW2 SW_SPDT, SW3 SW_SPDT, SW4 BUTTON, SW5 SW_SPDT, SW6 SW_SPDT, SW7 SW_SPDT, U1 SMF05CT1G, U2 M3406, U3 BQ21040DBVR, U4 SMF05CT1G, U5 QMC5883L, U6 BC805M, U7 LSM6DSV

Commit message: Bom consolidation UwU
Parts:
- added R29, R30, R31, R32: 200k, Patchwork Playground Footprints:R_0603_1608Metric, symbol Patchwork Playground Symbols:R_Small
- BT1, J4, J6, U6: now left out of the parts list
- C1, C2, C3, C4, C5, C7: MPN (none) -> C19666
- C10, C6, C9: MPN (none) -> C14663
- C8: MPN (none) -> C21120
- D1, D4: EXTENDED? (none) -> YES; MPN (none) -> C5178966
- D10, D11, D12, D13, D2, D3, D5, D7, D8, D9: MPN (none) -> C2290
- D6: EXTENDED? (none) -> YES; MPN (none) -> C965844
- J2: MPN (none) -> C165948
- L1: EXTENDED? (none) -> YES; MPN (none) -> C285966
- R1, R2: MPN (none) -> C23186
- R10, R11, R12, R13, R14, R15, R16, R17, R18, R19, R20, R21, R22, R25, R26, R27, R28, R3, R5, R6, R7, R8: MPN (none) -> C25804
- R23, R9: value 800k -> 200k; MPN (none) -> C25811
- R24: MPN (none) -> C25811
- R4: value 2M -> 200k; MPN (none) -> C25811
- SW1, SW2, SW3, SW5, SW6, SW7: EXTENDED? (none) -> YES; MPN (none) -> C2875122
- SW4: MPN (none) -> C318884
- U1, U4: MPN (none) -> C15879
- U2: EXTENDED? (none) -> YES; MPN (none) -> C83224
- U3: EXTENDED? (none) -> YES; MPN (none) -> C202311
- U5: EXTENDED? (none) -> YES; MPN (none) -> C976032
- U7: EXTENDED? (none) -> YES; MPN (none) -> C9900037528
Connections:
- net +3V3: now also R32.1; no longer R23.1
- net +BATT: now also R9.1; no longer R4.1
- net ADC: now also R4.1, R29.1, R30.2; no longer R4.2, R9.1
- net GND: now also R4.2, R29.2, R31.2; no longer R9.2
- net at R23.2, R24.1, U2.5 (FB): now also R31.1
- new net: R30.1, R9.2
- new net: R23.1, R32.2
Other:
- moved on the sheet: C3, C4, L1, R24

Commit message: prettify
Parts:
- renumbered C5 to C4, C4 to C5, R4 to R10, R29 to R11, R10 to R12, R11 to R13, R12 to R14, R13 to R15, R14 to R16, R15 to R17, R16 to R18, R17 to R19, R18 to R20, R19 to R21, R20 to R22, R21 to R23, R22 to R24, R24 to R25, R32 to R26, R23 to R27, R25 to R28, R26 to R29, R9 to R3, R31 to R30, R27 to R31, R28 to R32, R3 to R4, R30 to R5, R5 to R6, R6 to R7, R7 to R8, R8 to R9
Connections:
- net +BATT: now also R3.2; no longer R3.1
- net ADC: now also R10.2, R11.2, R5.1; no longer R10.1, R11.1, R5.2
- net GND: now also R10.1, R11.1; no longer R10.2, R11.2
- new net: R3.1, R5.2
Other:
- moved on the sheet: R10, R11, R27, R3, R5

Commit message: Removed some stuff from BOM owo
Parts:
- J1, J3, J5, TP1, TP10, TP11, TP12, TP2, TP3, TP4, TP5, TP6, TP7, TP8, TP9: now left out of the parts list
Changed lines of the file:
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@@
   )
   (symbol (lib_id "Patchwork Playground Symbols:Conn_01x02_Pin") (at 50.8 60.96 0) (unit 1)
-    (in_bom yes) (on_board yes) (dnp no)
+    (in_bom no) (on_board yes) (dnp no)
     (property "Reference" "J3" (at 50.8 58.42 0)
       (effects (font (size 1.27 1.27)))
@@
   )
   (symbol (lib_id "Patchwork Playground Symbols:TestPoint") (at 125.73 181.61 0) (unit 1)
-    (in_bom yes) (on_board yes) (dnp no)
+    (in_bom no) (on_board yes) (dnp no)
     (property "Reference" "TP4" (at 124.46 176.53 0)
       (effects (font (size 1.27 1.27)) (justify left))
@@
   )
   (symbol (lib_id "Patchwork Playground Symbols:TestPoint") (at 140.97 181.61 0) (unit 1)
-    (in_bom yes) (on_board yes) (dnp no)
+    (in_bom no) (on_board yes) (dnp no)
     (property "Reference" "TP7" (at 139.7 176.53 0)
       (effects (font (size 1.27 1.27)) (justify left))
@@
   )
   (symbol (lib_id "Patchwork Playground Symbols:TestPoint") (at 109.22 182.88 180) (unit 1)
-    (in_bom yes) (on_board yes) (dnp no)
+    (in_bom no) (on_board yes) (dnp no)
     (property "Reference" "TP1" (at 110.49 187.96 0)
       (effects (font (size 1.27 1.27)) (justify left))
@@
   )
   (symbol (lib_id "Patchwork Playground Symbols:TestPoint") (at 146.05 181.61 0) (unit 1)
-    (in_bom yes) (on_board yes) (dnp no)
+    (in_bom no) (on_board yes) (dnp no)
     (property "Reference" "TP8" (at 144.78 176.53 0)
       (effects (font (size 1.27 1.27)) (justify left))
@@
   )
   (symbol (lib_id "Patchwork Playground Symbols:TestPoint") (at 156.21 181.61 0) (unit 1)
-    (in_bom yes) (on_board yes) (dnp no)
+    (in_bom no) (on_board yes) (dnp no)
     (property "Reference" "TP10" (at 154.94 176.53 0)
       (effects (font (size 1.27 1.27)) (justify left))
@@
   )
   (symbol (lib_id "Patchwork Playground Symbols:TestPoint") (at 161.29 181.61 0) (unit 1)
-    (in_bom yes) (on_board yes) (dnp no)
+    (in_bom no) (on_board yes) (dnp no)
     (property "Reference" "TP11" (at 160.02 176.53 0)
       (effects (font (size 1.27 1.27)) (justify left))
@@
   )
   (symbol (lib_id "Patchwork Playground Symbols:TestPoint") (at 115.57 182.88 180) (unit 1)
-    (in_bom yes) (on_board yes) (dnp no)
+    (in_bom no) (on_board yes) (dnp no)
     (property "Reference" "TP2" (at 116.84 187.96 0)
       (effects (font (size 1.27 1.27)) (justify left))
@@
   )
   (symbol (lib_id "Patchwork Playground Symbols:TestPoint") (at 130.81 181.61 0) (unit 1)
-    (in_bom yes) (on_board yes) (dnp no)
+    (in_bom no) (on_board yes) (dnp no)
     (property "Reference" "TP5" (at 129.54 176.53 0)
       (effects (font (size 1.27 1.27)) (justify left))
@@
   )
   (symbol (lib_id "Patchwork Playground Symbols:TestPoint") (at 166.37 181.61 0) (unit 1)
-    (in_bom yes) (on_board yes) (dnp no)
+    (in_bom no) (on_board yes) (dnp no)
     (property "Reference" "TP12" (at 165.1 176.53 0)
       (effects (font (size 1.27 1.27)) (justify left))
@@
   )
   (symbol (lib_id "Patchwork Playground Symbols:Conn_01x02_Pin") (at 26.67 160.02 0) (unit 1)
-    (in_bom yes) (on_board yes) (dnp no)
+    (in_bom no) (on_board yes) (dnp no)
     (property "Reference" "J1" (at 26.67 157.48 0)
       (effects (font (size 1.27 1.27)))
@@
   )
   (symbol (lib_id "Patchwork Playground Symbols:TestPoint") (at 135.89 181.61 0) (unit 1)
-    (in_bom yes) (on_board yes) (dnp no)
+    (in_bom no) (on_board yes) (dnp no)
     (property "Reference" "TP6" (at 134.62 176.53 0)
       (effects (font (size 1.27 1.27)) (justify left))
@@
   )
   (symbol (lib_id "Patchwork Playground Symbols:TestPoint") (at 120.65 182.88 180) (unit 1)
-    (in_bom yes) (on_board yes) (dnp no)
+    (in_bom no) (on_board yes) (dnp no)
     (property "Reference" "TP3" (at 121.92 187.96 0)
       (effects (font (size 1.27 1.27)) (justify left))
@@
   )
   (symbol (lib_id "Patchwork Playground Symbols:TestPoint") (at 151.13 181.61 0) (unit 1)
-    (in_bom yes) (on_board yes) (dnp no)
+    (in_bom no) (on_board yes) (dnp no)
     (property "Reference" "TP9" (at 149.86 176.53 0)
       (effects (font (size 1.27 1.27)) (justify left))
@@
   )
   (symbol (lib_id "Patchwork Playground Symbols:Conn_01x02_Pin") (at 69.85 59.69 0) (unit 1)
-    (in_bom yes) (on_board yes) (dnp no)
+    (in_bom no) (on_board yes) (dnp no)
     (property "Reference" "J5" (at 69.85 57.15 0)
       (effects (font (size 1.27 1.27)))
